File: Controller/Controller.sch (EAGLE design)
At the start: 7 parts, among them U1 TPD4S009DBVR, U2 TPS2511DGN

Commit message: Modified controller
Parts:
- added JP2: (no value), adafruit:PINHD-1X3CB
- added U$1: SPARKFUN_USB_A, sparkfun-usb-a:SPARKFUN_USB_A
Connections:
- new net N$9: JP2.2, R2.1
- net N$1: now also U$1.USB+
- net N$2: now also U$1.USB-
- net N$3: now also JP2.1, U$1.USB_5V
- net N$4: now also JP2.3, U$1.USB_GND
Other:
- note removed: "DATA+"
- note removed: "DATA-"
- note removed: "GND"
- note removed: "VCC"
Changed lines of the file:
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@@
 <?xml version="1.0" encoding="utf-8"?>
 <!DOCTYPE eagle SYSTEM "eagle.dtd">
-<eagle version="7.0.0">
+<eagle version="7.1.0">
 <drawing>
 <settings>
@@
 <layer number="97" name="Info" color="7" fill="1" visible="yes" active="yes"/>
 <layer number="98" name="Guide" color="6" fill="1" visible="yes" active="yes"/>
+<layer number="99" name="SpiceOrder" color="7" fill="1" visible="yes" active="yes"/>
 <layer number="100" name="Muster" color="7" fill="1" visible="no" active="no"/>
 <layer number="101" name="Patch_Top" color="12" fill="4" visible="yes" active="yes"/>
@@
 <layer number="111" name="LPC17xx" color="7" fill="1" visible="yes" active="yes"/>
 <layer number="112" name="tSilk" color="7" fill="1" visible="yes" active="yes"/>
+<layer number="113" name="IDFDebug" color="4" fill="1" visible="yes" active="yes"/>
 <layer number="116" name="Patch_BOT" color="9" fill="4" visible="yes" active="yes"/>
 <layer number="121" name="_tsilk" color="7" fill="1" visible="yes" active="yes"/>
@@
 <part name="C2" library="adafruit" deviceset="CPOL-US" device="E2-5"/>
 <part name="R2" library="SparkFun-Passives" deviceset="RESISTOR" device="KIT"/>
+<part name="U$1" library="sparkfun-usb-a" deviceset="SPARKFUN_USB_A" device=""/>
+<part name="JP2" library="adafruit" deviceset="PINHD-1X3" device="CB"/>
 </parts>
 <sheets>
 <sheet>
 <plain>
-<text x="76.2" y="38.1" size="1.778" layer="91">GND</text>
-<text x="55.88" y="38.1" size="1.778" layer="91">VCC</text>
-<text x="68.58" y="38.1" size="1.778" layer="91">DATA+</text>
-<text x="60.96" y="38.1" size="1.778" layer="91">DATA-</text>
-<rectangle x1="55.88" y1="30.48" x2="81.28" y2="40.64" layer="95"/>
 </plain>
 <instances>
@@
 <instance part="C2" gate="G$1" x="119.38" y="73.66"/>
 <instance part="R2" gate="G$1" x="185.42" y="132.08" rot="R180"/>
+<instance part="U$1" gate="G$1" x="68.58" y="17.78" rot="R90"/>
+<instance part="JP2" gate="A" x="203.2" y="132.08"/>
 </instances>
 <busses>
@@
 <wire x1="88.9" y1="50.8" x2="73.66" y2="50.8" width="0.1524" layer="91"/>
 <wire x1="73.66" y1="50.8" x2="73.66" y2="40.64" width="0.1524" layer="91"/>
+<pinref part="U$1" gate="G$1" pin="USB+"/>
+<wire x1="73.66" y1="40.64" x2="71.12" y2="40.64" width="0.1524" layer="91"/>
+<wire x1="71.12" y1="40.64" x2="71.12" y2="27.94" width="0.1524" layer="91"/>
 </segment>
 </net>
@@
 <segment>
 <wire x1="91.44" y1="53.34" x2="63.5" y2="53.34" width="0.1524" layer="91"/>
-<wire x1="63.5" y1="53.34" x2="63.5" y2="40.64" width="0.1524" layer="91"/>
+<wire x1="63.5" y1="53.34" x2="63.5" y2="35.56" width="0.1524" layer="91"/>
 <pinref part="U1" gate="A" pin="D1+"/>
 <wire x1="81.28" y1="137.16" x2="91.44" y2="137.16" width="0.1524" layer="91"/>
 <wire x1="91.44" y1="137.16" x2="91.44" y2="53.34" width="0.1524" layer="91"/>
+<pinref part="U$1" gate="G$1" pin="USB-"/>
+<wire x1="63.5" y1="35.56" x2="73.66" y2="35.56" width="0.1524" layer="91"/>
+<wire x1="73.66" y1="35.56" x2="73.66" y2="27.94" width="0.1524" layer="91"/>
 </segment>
 </net>
 <net name="N$3" class="0">
 <segment>
-<pinref part="U1" gate="A" pin="VCC"/>
-<wire x1="45.72" y1="137.16" x2="43.18" y2="137.16" width="0.1524" layer="91"/>
-<wire x1="43.18" y1="137.16" x2="35.56" y2="137.16" width="0.1524" layer="91"/>
-<wire x1="35.56" y1="137.16" x2="35.56" y2="53.34" width="0.1524" layer="91"/>
-<wire x1="35.56" y1="53.34" x2="58.42" y2="53.34" width="0.1524" layer="91"/>
-<wire x1="58.42" y1="53.34" x2="58.42" y2="40.64" width="0.1524" layer="91"/>
-<wire x1="43.18" y1="137.16" x2="43.18" y2="157.48" width="0.1524" layer="91"/>
-<wire x1="43.18" y1="157.48" x2="114.3" y2="157.48" width="0.1524" layer="91"/>
+<wire x1="35.56" y1="157.48" x2="114.3" y2="157.48" width="0.1524" layer="91"/>
 <wire x1="114.3" y1="157.48" x2="165.1" y2="157.48" width="0.1524" layer="91"/>
 <wire x1="165.1" y1="157.48" x2="165.1" y2="137.16" width="0.1524" layer="91"/>
@@
 <wire x1="119.38" y1="88.9" x2="119.38" y2="76.2" width="0.1524" layer="91"/>
 <pinref part="C2" gate="G$1" pin="+"/>
+<pinref part="U$1" gate="G$1" pin="USB_5V"/>
+<pinref part="U1" gate="A" pin="VCC"/>
+<wire x1="45.72" y1="137.16" x2="35.56" y2="137.16" width="0.1524" layer="91"/>
+<wire x1="35.56" y1="137.16" x2="35.56" y2="53.34" width="0.1524" layer="91"/>
+<wire x1="35.56" y1="53.34" x2="58.42" y2="53.34" width="0.1524" layer="91"/>
+<wire x1="58.42" y1="53.34" x2="58.42" y2="27.94" width="0.1524" layer="91"/>
+<wire x1="58.42" y1="27.94" x2="63.5" y2="27.94" width="0.1524" layer="91"/>
+<wire x1="35.56" y1="157.48" x2="35.56" y2="137.16" width="0.1524" layer="91"/>
+<junction x="35.56" y="137.16"/>
+<wire x1="165.1" y1="137.16" x2="190.5" y2="137.16" width="0.1524" layer="91"/>
+<wire x1="190.5" y1="137.16" x2="193.04" y2="134.62" width="0.1524" layer="91"/>
+<pinref part="JP2" gate="A" pin="1"/>
+<wire x1="193.04" y1="134.62" x2="200.66" y2="134.62" width="0.1524" layer="91"/>
 </segment>
 </net>
 <net name="N$4" class="0">
 <segment>
-<wire x1="78.74" y1="55.88" x2="78.74" y2="40.64" width="0.1524" layer="91"/>
+<wire x1="78.74" y1="55.88" x2="78.74" y2="33.02" width="0.1524" layer="91"/>
 <wire x1="165.1" y1="55.88" x2="119.38" y2="55.88" width="0.1524" layer="91"/>
 <junction x="78.74" y="55.88"/>
@@
 <wire x1="40.64" y1="55.88" x2="78.74" y2="55.88" width="0.1524" layer="91"/>
 <pinref part="C1" gate="G$1" pin="-"/>
-<wire x1="165.1" y1="111.76" x2="165.1" y2="55.88" width="0.1524" layer="91"/>
+<wire x1="165.1" y1="111.76" x2="165.1" y2="104.14" width="0.1524" layer="91"/>
 <pinref part="U2" gate="A" pin="GND"/>
+<wire x1="165.1" y1="104.14" x2="165.1" y2="55.88" width="0.1524" layer="91"/>
 <wire x1="124.46" y1="109.22" x2="106.68" y2="109.22" width="0.1524" layer="91"/>
 <wire x1="106.68" y1="109.22" x2="106.68" y2="55.88" width="0.1524" layer="91"/>
@@
 <wire x1="119.38" y1="68.58" x2="119.38" y2="55.88" width="0.1524" layer="91"/>
 <junction x="119.38" y="55.88"/>
+<pinref part="U$1" gate="G$1" pin="USB_GND"/>
+<wire x1="78.74" y1="33.02" x2="66.04" y2="33.02" width="0.1524" layer="91"/>
+<wire x1="66.04" y1="33.02" x2="66.04" y2="27.94" width="0.1524" layer="91"/>
+<wire x1="165.1" y1="104.14" x2="167.64" y2="104.14" width="0.1524" layer="91"/>
+<wire x1="167.64" y1="104.14" x2="193.04" y2="129.54" width="0.1524" layer="91"/>
+<junction x="165.1" y="104.14"/>
+<pinref part="JP2" gate="A" pin="3"/>
+<wire x1="193.04" y1="129.54" x2="200.66" y2="129.54" width="0.1524" layer="91"/>
 </segment>
 </net>
@@
 </segment>
 </net>
+<net name="N$9" class="0">
+<segment>
+<pinref part="R2" gate="G$1" pin="1"/>
+<pinref part="JP2" gate="A" pin="2"/>
+<wire x1="190.5" y1="132.08" x2="200.66" y2="132.08" width="0.1524" layer="91"/>
+</segment>
+</net>
