File: Solar Charger (Through-Hole)/Solar USB.sch (EAGLE design)
At the start: 22 parts, among them U1 MCP73871-2CCI/ML

Commit message: boost
Parts:
- removed U1: MCP73871-2CCI/ML, Microchip_By_element14_Batch_1:MCP73871-2CCI/ML
- added IC1: MCP73871, adafruit:MCP73871
- C1, C2, C4: device SparkFun-Capacitors:10UF-25V-20%(PTH)KIT -> adafruit:CPOL-USE2.5-5
- C3: device SparkFun-Capacitors:10UF-25V-20%(PTH)KIT -> adafruit:CPOL-USE7.5-16
- JP1, JP2, JP3: value M023.5MM -> M02PTH; device SparkFun-Connectors:M023.5MM -> SparkFun-Connectors:M02PTH
Connections:
- removed net N$6: C1.+, JP3.1, U1.VBAT, U1.VBAT_2, U1.VBAT_SENSE
- removed net N$7: C2.+, JP2.1, U1.OUT, U1.OUT_2
- new net N$15: C2.+, IC1.OUT1, IC1.OUT2, JP2.1
- new net N$17: C1.+, IC1.VBAT1, IC1.VBAT2, IC1.VBAT3, JP3.1
- net N$1: now also IC1./PG, LED3.C; no longer R9.2, U1.THERM
- net N$10: now also IC1./TE, IC1.CE, IC1.IN1, IC1.IN2, IC1.PROG2, IC1.SEL; no longer U1.*TE, U1.CE, U1.IN, U1.IN_2, U1.PROG2, U1.SEL
- net N$11: now also IC1.THERM, R9.2; no longer LED1.C, U1.STAT1/*LBO
- net N$16: now also IC1.VPCC; no longer U1.VPCC
- net N$2: now also IC1.GND1, IC1.GND2, IC1.GND3; no longer U1.EP, U1.VSS, U1.VSS_2
- net N$3: now also IC1.PROG3; no longer U1.PROG3
- net N$4: now also IC1.PROG1; no longer U1.PROG1
- net N$8: now also IC1.STAT2, LED2.C; no longer LED3.C, U1.*PG
- net N$9: now also IC1.STAT1/LBO, LED1.C; no longer LED2.C, U1.STAT2
Other:
- moved on the sheet: R4, R5, R8, R9, THERM

Commit message: Made some changes to feedback loop and reorganized controller
Parts:
- JP1, JP2, JP3: value M02PTH -> M023.5MM; device SparkFun-Connectors:M02PTH -> SparkFun-Connectors:M023.5MM
- R1, R2, R3, R4, R5, R6, R7, R8, R9, THERM: device SparkFun-Resistors:1KOHM1/4W5%(PTH) -> adafruit:R-US_0207/10
Changed lines of the file:
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@@
 <parts>
 <part name="FRAME1" library="SparkFun-Aesthetics" deviceset="FRAME-LETTER" device=""/>
-<part name="JP1" library="SparkFun-Connectors" deviceset="M02" device="PTH" value="M02PTH"/>
-<part name="JP2" library="SparkFun-Connectors" deviceset="M02" device="PTH" value="M02PTH"/>
-<part name="JP3" library="SparkFun-Connectors" deviceset="M02" device="PTH" value="M02PTH"/>
+<part name="JP1" library="SparkFun-Connectors" deviceset="M02" device="3.5MM" value="M023.5MM"/>
+<part name="JP2" library="SparkFun-Connectors" deviceset="M02" device="3.5MM" value="M023.5MM"/>
+<part name="JP3" library="SparkFun-Connectors" deviceset="M02" device="3.5MM" value="M023.5MM"/>
 <part name="C1" library="adafruit" deviceset="CPOL-US" device="E2.5-5" value="10uF"/>
 <part name="C2" library="adafruit" deviceset="CPOL-US" device="E2.5-5" value="10uF"/>
@@
 <part name="LED2" library="SparkFun-LED" deviceset="LED" device="5MM"/>
 <part name="LED3" library="SparkFun-LED" deviceset="LED" device="5MM"/>
-<part name="R1" library="SparkFun-Resistors" deviceset="1KOHM1/4W5%(PTH)" device=""/>
-<part name="R2" library="SparkFun-Resistors" deviceset="1KOHM1/4W5%(PTH)" device=""/>
-<part name="R3" library="SparkFun-Resistors" deviceset="1KOHM1/4W5%(PTH)" device=""/>
-<part name="R4" library="SparkFun-Resistors" deviceset="1KOHM1/4W5%(PTH)" device="" value="100k"/>
-<part name="R5" library="SparkFun-Resistors" deviceset="1KOHM1/4W5%(PTH)" device="" value="1k"/>
-<part name="R6" library="SparkFun-Resistors" deviceset="1KOHM1/4W5%(PTH)" device="" value="270k"/>
-<part name="R7" library="SparkFun-Resistors" deviceset="1KOHM1/4W5%(PTH)" device="" value="100k"/>
-<part name="THERM" library="SparkFun-Resistors" deviceset="1KOHM1/4W5%(PTH)" device="" value="10k"/>
-<part name="R8" library="SparkFun-Resistors" deviceset="1KOHM1/4W5%(PTH)" device="" value="150k"/>
-<part name="R9" library="SparkFun-Resistors" deviceset="1KOHM1/4W5%(PTH)" device="" value="1k"/>
+<part name="R1" library="adafruit" deviceset="R-US_" device="0207/10"/>
+<part name="R2" library="adafruit" deviceset="R-US_" device="0207/10"/>
+<part name="R3" library="adafruit" deviceset="R-US_" device="0207/10"/>
+<part name="R4" library="adafruit" deviceset="R-US_" device="0207/10" value="100k"/>
+<part name="R5" library="adafruit" deviceset="R-US_" device="0207/10" value="1k"/>
+<part name="R6" library="adafruit" deviceset="R-US_" device="0207/10" value="270k"/>
+<part name="R7" library="adafruit" deviceset="R-US_" device="0207/10" value="100k"/>
+<part name="THERM" library="adafruit" deviceset="R-US_" device="0207/10" value="10k"/>
+<part name="R8" library="adafruit" deviceset="R-US_" device="0207/10" value="150k"/>
+<part name="R9" library="adafruit" deviceset="R-US_" device="0207/10" value="1k"/>
 <part name="C3" library="adafruit" deviceset="CPOL-US" device="E7.5-16" value="4700uF"/>
 <part name="C4" library="adafruit" deviceset="CPOL-US" device="E2.5-5" value="10uF"/>
