File: Final/Final.sch (EAGLE design)
At the start: 27 parts, among them IC1 MCP73871, J1 POWER_JACKPTH, U1 TPS2561DRCT, U2 TPS61030PWPR

Commit message: wired final solar
Changed lines of the file:
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@@
-</segment>
-</net>
-<net name="N$8" class="0">
-<segment>
-<pinref part="IC1" gate="G$1" pin="/PG"/>
-<pinref part="PWR" gate="G$1" pin="C"/>
-<wire x1="86.36" y1="147.32" x2="73.66" y2="147.32" width="0.1524" layer="91"/>
-</segment>
-</net>
-<net name="N$9" class="0">
-<segment>
-<pinref part="IC1" gate="G$1" pin="STAT2"/>
-<pinref part="DONE" gate="G$1" pin="C"/>
-<wire x1="86.36" y1="144.78" x2="66.04" y2="144.78" width="0.1524" layer="91"/>
-<wire x1="66.04" y1="144.78" x2="66.04" y2="152.4" width="0.1524" layer="91"/>
 </segment>
 </net>
 <net name="N$10" class="0">
 <segment>
+<pinref part="CHRG" gate="G$1" pin="C"/>
+<wire x1="58.42" y1="142.24" x2="58.42" y2="157.48" width="0.1524" layer="91"/>
 <pinref part="IC1" gate="G$1" pin="STAT1/LBO"/>
-<pinref part="CHRG" gate="G$1" pin="C"/>
-<wire x1="86.36" y1="142.24" x2="58.42" y2="142.24" width="0.1524" layer="91"/>
-<wire x1="58.42" y1="142.24" x2="58.42" y2="157.48" width="0.1524" layer="91"/>
+<wire x1="58.42" y1="142.24" x2="86.36" y2="142.24" width="0.1524" layer="91"/>
 </segment>
 </net>
@@
 </segment>
 </net>
+<net name="N$9" class="0">
+<segment>
+<pinref part="DONE" gate="G$1" pin="C"/>
+<wire x1="66.04" y1="152.4" x2="66.04" y2="144.78" width="0.1524" layer="91"/>
+<pinref part="IC1" gate="G$1" pin="STAT2"/>
+<wire x1="66.04" y1="144.78" x2="86.36" y2="144.78" width="0.1524" layer="91"/>
+</segment>
+</net>
+<net name="N$14" class="0">
+<segment>
+<pinref part="PWR" gate="G$1" pin="C"/>
+<pinref part="IC1" gate="G$1" pin="/PG"/>
+<wire x1="86.36" y1="147.32" x2="73.66" y2="147.32" width="0.1524" layer="91"/>
+</segment>
+</net>

Commit message: wired up solar board
Parts:
- FRAME1: value FRAME-LETTER -> FRAME-LEDGER; device SparkFun-Aesthetics:FRAME-LETTER -> SparkFun-Aesthetics:FRAME-LEDGER
Connections:
- net N$16 renamed V_BATT
Other:
- moved on the sheet: BATT, C1, C2, C3, C4, CHRG, D1, DONE, J1, PWR, R1, R10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

Commit message: wired boost sch and brd
Parts:
- added 5V, LOW: (no value), adafruit:LED5MM
- added C5: 10 uF, adafruit:CPOL-USE2.5-5
- added C6: 0.1 uF, adafruit:CPOL-USE2.5-5
- added C7: 2.2 uF, adafruit:CPOL-USE2.5-5
- added C8, C9: 100 uF, adafruit:CPOL-USE2.5-5
- added L1: 6.8 uH, rcl:L-USLAL03
- added MMUN2133L1G: BC847C-7-F, Diodes_Inc_By_element14_Batch_1:BC847C-7-F
- added R11, R13: 1.87 MOhm, adafruit:R-US_0207/10
- added R12: 200 kOhm, adafruit:R-US_0207/10
- added R14: 340 kOhm, adafruit:R-US_0207/10
- added R15, R16: (no value), adafruit:R-US_0207/10
- added R17: 24.9 kOhm, adafruit:R-US_0207/10
- added R8: 1 kOhm, adafruit:R-US_0207/10
- R10: value 150 kOhm -> 200 kOhm
- R9: value 1 kOhm -> 150 kOhm
Connections:
- new net 5V: C7.+, C8.+, C9.+, R11.1, R15.1, U1.IN, U1.IN_2, U2.VOUT, U2.VOUT_2, U2.VOUT_3
- new net N$15: R13.2, R14.1, U2.LBI
- new net N$16: R11.2, R12.1, U2.FB
- new net N$17: 5V.A, R15.2
- new net N$18: L1.1, U2.SW, U2.SW_2
- new net N$19: R10.2, U2.EN
- new net N$20: MMUN2133L1G.B, U2.LBO
- new net N$21: R17.1, U1.ILIM
- new net N$22: MMUN2133L1G.C, R16.1
- new net N$23: LOW.A, R16.2
- new net N$24: U1.EN1, U1.EN2
- net GND: now also 5V.C, C5.-, C6.-, C7.-, C8.-, C9.-, LOW.C, R12.2, R14.2, R17.2, R9.2, U1.EPAD, U1.GND, U2.GND, U2.PGND, U2.PGND_2, U2.PGND_3, U2.POWERPAD, U2.SYNC; no longer R10.2
- net N$12: now also R8.1; no longer R9.1
- net N$13: now also R8.2, R9.1; no longer R10.1, R9.2
- net V_BATT: now also C5.+, C6.+, L1.2, MMUN2133L1G.E, R10.1, R13.1, U2.VBAT
Other:
- moved on the sheet: R10, R9

Commit message: DONE!!!!
Parts:
- added C10: 0.1 uF, adafruit:CPOL-USE2.5-5
- added C11: 150 uF, adafruit:CPOL-USE2.5-5
- added R19: 100 kOhm, adafruit:R-US_0207/10
Connections:
- removed net N$24: U1.EN1, U1.EN2
- new net N$26: R19.1, U1.~FAULT1
- new net N$27: C11.+, U$1.VBUS, U1.OUT1
- new net N$29: TPS2513.P$1, U$1.D+
- new net N$30: TPS2513.P$6, U$1.D-
- net 5V: now also C10.+, R19.2, TPS2513.P$5; no longer U1.IN_2
- net GND: now also C10.-, C11.-, TPS2513.P$2, U$1.GND
Other:
- moved on the sheet: R17, TPS2513, U1
Changed lines of the file:
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@@
 <part name="R17" library="adafruit" deviceset="R-US_" device="0207/10" value="24.9 kOhm"/>
 <part name="GND15" library="SparkFun-Aesthetics" deviceset="GND" device=""/>
+<part name="SUPPLY13" library="SparkFun-Aesthetics" deviceset="5V" device=""/>
+<part name="R19" library="adafruit" deviceset="R-US_" device="0207/10" value="100 kOhm"/>
+<part name="C10" library="adafruit" deviceset="CPOL-US" device="E2.5-5" value="0.1 uF"/>
+<part name="GND16" library="SparkFun-Aesthetics" deviceset="GND" device=""/>
+<part name="C11" library="adafruit" deviceset="CPOL-US" device="E2.5-5" value="150 uF"/>
+<part name="GND17" library="SparkFun-Aesthetics" deviceset="GND" device=""/>
+<part name="SUPPLY14" library="SparkFun-Aesthetics" deviceset="5V" device=""/>
+<part name="GND18" library="SparkFun-Aesthetics" deviceset="GND" device=""/>
+<part name="GND19" library="SparkFun-Aesthetics" deviceset="GND" device=""/>
 </parts>
 <sheets>
@@
 <instance part="FRAME1" gate="G$1" x="0" y="0"/>
 <instance part="FRAME1" gate="G$2" x="330.2" y="0"/>
-<instance part="U1" gate="A" x="99.06" y="101.6"/>
-<instance part="TPS2513" gate="G$1" x="99.06" y="48.26"/>
+<instance part="U1" gate="A" x="99.06" y="73.66"/>
+<instance part="TPS2513" gate="G$1" x="320.04" y="132.08"/>
 <instance part="U2" gate="A" x="317.5" y="203.2"/>
 <instance part="IC1" gate="G$1" x="129.54" y="200.66"/>
 <instance part="U3" gate="G$1" x="7.62" y="241.3" rot="R180"/>
 <instance part="J1" gate="G$1" x="15.24" y="256.54"/>
-<instance part="U$1" gate="G$1" x="314.96" y="86.36"/>
+<instance part="U$1" gate="G$1" x="314.96" y="68.58"/>
 <instance part="D1" gate="G$1" x="25.4" y="264.16"/>
 <instance part="C1" gate="G$1" x="35.56" y="259.08"/>
@@
 <instance part="LOW" gate="G$1" x="401.32" y="246.38"/>
 <instance part="GND13" gate="1" x="401.32" y="233.68"/>
-<instance part="SUPPLY12" gate="G$1" x="33.02" y="121.92"/>
-<instance part="GND14" gate="1" x="63.5" y="71.12"/>
-<instance part="R17" gate="G$1" x="134.62" y="83.82" rot="R270"/>
-<instance part="GND15" gate="1" x="134.62" y="71.12"/>
+<instance part="SUPPLY12" gate="G$1" x="33.02" y="93.98"/>
+<instance part="GND14" gate="1" x="63.5" y="43.18"/>
+<instance part="R17" gate="G$1" x="134.62" y="55.88" rot="R270"/>
+<instance part="GND15" gate="1" x="134.62" y="43.18"/>
+<instance part="SUPPLY13" gate="G$1" x="177.8" y="71.12"/>
+<instance part="R19" gate="G$1" x="154.94" y="53.34"/>
+<instance part="C10" gate="G$1" x="33.02" y="81.28"/>
+<instance part="GND16" gate="1" x="33.02" y="71.12"/>
+<instance part="C11" gate="G$1" x="142.24" y="88.9"/>
+<instance part="GND17" gate="1" x="142.24" y="78.74"/>
+<instance part="SUPPLY14" gate="G$1" x="363.22" y="142.24"/>
+<instance part="GND18" gate="1" x="266.7" y="116.84"/>
+<instance part="GND19" gate="1" x="281.94" y="50.8"/>
 </instances>
 <busses>
@@
 <segment>
 <pinref part="U1" gate="A" pin="GND"/>
-<wire x1="68.58" y1="91.44" x2="66.04" y2="91.44" width="0.1524" layer="91"/>
-<wire x1="66.04" y1="91.44" x2="66.04" y2="88.9" width="0.1524" layer="91"/>
+<wire x1="68.58" y1="63.5" x2="66.04" y2="63.5" width="0.1524" layer="91"/>
+<wire x1="66.04" y1="63.5" x2="66.04" y2="60.96" width="0.1524" layer="91"/>
 <pinref part="U1" gate="A" pin="EPAD"/>
-<wire x1="66.04" y1="88.9" x2="68.58" y2="88.9" width="0.1524" layer="91"/>
-<wire x1="66.04" y1="88.9" x2="63.5" y2="88.9" width="0.1524" layer="91"/>
-<junction x="66.04" y="88.9"/>
+<wire x1="66.04" y1="60.96" x2="68.58" y2="60.96" width="0.1524" layer="91"/>
+<wire x1="66.04" y1="60.96" x2="63.5" y2="60.96" width="0.1524" layer="91"/>
+<junction x="66.04" y="60.96"/>
 <pinref part="GND14" gate="1" pin="GND"/>
-<wire x1="63.5" y1="88.9" x2="63.5" y2="73.66" width="0.1524" layer="91"/>
+<wire x1="63.5" y1="60.96" x2="63.5" y2="45.72" width="0.1524" layer="91"/>
 </segment>
 <segment>
 <pinref part="R17" gate="G$1" pin="2"/>
 <pinref part="GND15" gate="1" pin="GND"/>
-<wire x1="134.62" y1="78.74" x2="134.62" y2="73.66" width="0.1524" layer="91"/>
+<wire x1="134.62" y1="50.8" x2="134.62" y2="45.72" width="0.1524" layer="91"/>
+</segment>
+<segment>
+<pinref part="C10" gate="G$1" pin="-"/>
+<pinref part="GND16" gate="1" pin="GND"/>
+<wire x1="33.02" y1="73.66" x2="33.02" y2="76.2" width="0.1524" layer="91"/>
+</segment>
+<segment>
+<pinref part="TPS2513" gate="G$1" pin="P$2"/>
+<pinref part="GND18" gate="1" pin="GND"/>
+<wire x1="299.72" y1="127" x2="266.7" y2="127" width="0.1524" layer="91"/>
+<wire x1="266.7" y1="127" x2="266.7" y2="119.38" width="0.1524" layer="91"/>
+</segment>
+<segment>
+<pinref part="GND19" gate="1" pin="GND"/>
+<wire x1="281.94" y1="68.58" x2="281.94" y2="53.34" width="0.1524" layer="91"/>
+<pinref part="U$1" gate="G$1" pin="GND"/>
+<wire x1="312.42" y1="68.58" x2="281.94" y2="68.58" width="0.1524" layer="91"/>
+</segment>
+<segment>
+<pinref part="C11" gate="G$1" pin="-"/>
+<pinref part="GND17" gate="1" pin="GND"/>
+<wire x1="142.24" y1="83.82" x2="142.24" y2="81.28" width="0.1524" layer="91"/>
 </segment>
 </net>
@@
 </segment>
 <segment>
+<pinref part="SUPPLY13" gate="G$1" pin="5V"/>
+<wire x1="177.8" y1="53.34" x2="177.8" y2="71.12" width="0.1524" layer="91"/>
+<pinref part="R19" gate="G$1" pin="2"/>
+<wire x1="160.02" y1="53.34" x2="177.8" y2="53.34" width="0.1524" layer="91"/>
+</segment>
+<segment>
+<pinref part="C10" gate="G$1" pin="+"/>
 <pinref part="SUPPLY12" gate="G$1" pin="5V"/>
-<wire x1="33.02" y1="121.92" x2="33.02" y2="106.68" width="0.1524" layer="91"/>
-<pinref part="U1" gate="A" pin="IN_2"/>
-<wire x1="68.58" y1="106.68" x2="66.04" y2="106.68" width="0.1524" layer="91"/>
+<wire x1="33.02" y1="83.82" x2="33.02" y2="88.9" width="0.1524" layer="91"/>
+<wire x1="33.02" y1="88.9" x2="33.02" y2="93.98" width="0.1524" layer="91"/>
+<wire x1="48.26" y1="76.2" x2="48.26" y2="88.9" width="0.1524" layer="91"/>
+<wire x1="48.26" y1="88.9" x2="33.02" y2="88.9" width="0.1524" layer="91"/>
+<junction x="33.02" y="88.9"/>
 <pinref part="U1" gate="A" pin="IN"/>
-<wire x1="66.04" y1="106.68" x2="33.02" y2="106.68" width="0.1524" layer="91"/>
-<wire x1="68.58" y1="104.14" x2="66.04" y2="104.14" width="0.1524" layer="91"/>
-<wire x1="66.04" y1="104.14" x2="66.04" y2="106.68" width="0.1524" layer="91"/>
-<junction x="66.04" y="106.68"/>
+<wire x1="68.58" y1="76.2" x2="48.26" y2="76.2" width="0.1524" layer="91"/>
+</segment>
+<segment>
+<pinref part="TPS2513" gate="G$1" pin="P$5"/>
+<pinref part="SUPPLY14" gate="G$1" pin="5V"/>
+<wire x1="340.36" y1="127" x2="363.22" y2="127" width="0.1524" layer="91"/>
+<wire x1="363.22" y1="127" x2="363.22" y2="142.24" width="0.1524" layer="91"/>
 </segment>
 </net>
@@
 </segment>
 </net>
-<net name="N$24" class="0">
-<segment>
-<pinref part="U1" gate="A" pin="EN2"/>
-<wire x1="68.58" y1="96.52" x2="66.04" y2="96.52" width="0.1524" layer="91"/>
-<wire x1="66.04" y1="96.52" x2="66.04" y2="99.06" width="0.1524" layer="91"/>
-<pinref part="U1" gate="A" pin="EN1"/>
-<wire x1="66.04" y1="99.06" x2="68.58" y2="99.06" width="0.1524" layer="91"/>
-</segment>
-</net>
 <net name="N$21" class="0">
 <segment>
 <pinref part="U1" gate="A" pin="ILIM"/>
 <pinref part="R17" gate="G$1" pin="1"/>
-<wire x1="129.54" y1="88.9" x2="134.62" y2="88.9" width="0.1524" layer="91"/>
-</segment>
-</net>
+<wire x1="129.54" y1="60.96" x2="134.62" y2="60.96" width="0.1524" layer="91"/>
+</segment>
+</net>
+<net name="N$26" class="0">
+<segment>
+<pinref part="U1" gate="A" pin="~FAULT1"/>
+<wire x1="129.54" y1="63.5" x2="142.24" y2="63.5" width="0.1524" layer="91"/>
+<wire x1="142.24" y1="63.5" x2="142.24" y2="53.34" width="0.1524" layer="91"/>
+<pinref part="R19" gate="G$1" pin="1"/>
+<wire x1="142.24" y1="53.34" x2="149.86" y2="53.34" width="0.1524" layer="91"/>
+</segment>
+</net>
+<net name="N$27" class="0">
+<segment>
+<pinref part="U1" gate="A" pin="OUT1"/>
+<wire x1="129.54" y1="68.58" x2="137.16" y2="68.58" width="0.1524" layer="91"/>
+<wire x1="137.16" y1="68.58" x2="137.16" y2="96.52" width="0.1524" layer="91"/>
+<pinref part="C11" gate="G$1" pin="+"/>
+<wire x1="137.16" y1="96.52" x2="142.24" y2="96.52" width="0.1524" layer="91"/>
+<wire x1="142.24" y1="96.52" x2="142.24" y2="91.44" width="0.1524" layer="91"/>
+<wire x1="142.24" y1="96.52" x2="185.42" y2="96.52" width="0.1524" layer="91"/>
+<junction x="142.24" y="96.52"/>
+<pinref part="U$1" gate="G$1" pin="VBUS"/>
+<wire x1="312.42" y1="71.12" x2="185.42" y2="71.12" width="0.1524" layer="91"/>
+<wire x1="185.42" y1="71.12" x2="185.42" y2="96.52" width="0.1524" layer="91"/>
+</segment>
+</net>
+<net name="N$29" class="0">
+<segment>
+<pinref part="TPS2513" gate="G$1" pin="P$1"/>
+<wire x1="299.72" y1="132.08" x2="256.54" y2="132.08" width="0.1524" layer="91"/>
+<wire x1="256.54" y1="132.08" x2="256.54" y2="76.2" width="0.1524" layer="91"/>
+<pinref part="U$1" gate="G$1" pin="D+"/>
+<wire x1="256.54" y1="76.2" x2="312.42" y2="76.2" width="0.1524" layer="91"/>
+</segment>
+</net>
+<net name="N$30" class="0">
+<segment>
+<pinref part="TPS2513" gate="G$1" pin="P$6"/>
+<wire x1="340.36" y1="132.08" x2="345.44" y2="132.08" width="0.1524" layer="91"/>
+<wire x1="345.44" y1="132.08" x2="345.44" y2="149.86" width="0.1524" layer="91"/>
+<wire x1="345.44" y1="149.86" x2="251.46" y2="149.86" width="0.1524" layer="91"/>
+<wire x1="251.46" y1="149.86" x2="251.46" y2="73.66" width="0.1524" layer="91"/>
+<pinref part="U$1" gate="G$1" pin="D-"/>
+<wire x1="251.46" y1="73.66" x2="312.42" y2="73.66" width="0.1524" layer="91"/>
+</segment>
+</net>

Commit message: Made even more tweeks to the design
Parts:
- U3: value (none) -> USB-MICROB; device SparkFun-Connectors:USB-ABCONN-11794 -> SparkFun-Connectors:USB-MICROB
Changed lines of the file:
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@@
 <part name="U2" library="TPS61230" deviceset="TPS61030PWPR" device=""/>
 <part name="IC1" library="adafruit" deviceset="MCP73871" device=""/>
-<part name="U3" library="SparkFun-Connectors" deviceset="USB-AB" device="CONN-11794"/>
+<part name="U3" library="SparkFun-Connectors" deviceset="USB" device="-MICROB"/>
 <part name="J1" library="SparkFun-Connectors" deviceset="POWER_JACK" device="PTH"/>
 <part name="U$1" library="SparkFun-Connectors" deviceset="USB+SHIELD" device="USB-A-S-NOSILK-FEMALE"/>
@@
 <instance part="U2" gate="A" x="317.5" y="203.2"/>
 <instance part="IC1" gate="G$1" x="129.54" y="200.66"/>
-<instance part="U3" gate="G$1" x="7.62" y="241.3" rot="R180"/>
+<instance part="U3" gate="G$1" x="10.16" y="246.38" rot="R180"/>
 <instance part="J1" gate="G$1" x="15.24" y="256.54"/>
 <instance part="U$1" gate="G$1" x="314.96" y="68.58"/>
@@
 </segment>
 <segment>
-<pinref part="U3" gate="G$1" pin="GND"/>
-<pinref part="GND2" gate="1" pin="GND"/>
-<wire x1="12.7" y1="236.22" x2="22.86" y2="236.22" width="0.1524" layer="91"/>
-</segment>
-<segment>
 <pinref part="GND4" gate="1" pin="GND"/>
 <pinref part="R5" gate="G$1" pin="1"/>
@@
 <wire x1="142.24" y1="83.82" x2="142.24" y2="81.28" width="0.1524" layer="91"/>
 </segment>
+<segment>
+<pinref part="U3" gate="G$1" pin="GND"/>
+<pinref part="GND2" gate="1" pin="GND"/>
+<wire x1="12.7" y1="238.76" x2="22.86" y2="238.76" width="0.1524" layer="91"/>
+<wire x1="22.86" y1="238.76" x2="22.86" y2="236.22" width="0.1524" layer="91"/>
+</segment>
 </net>

Commit message: more tweeks
Parts:
- renumbered R19 to R18
Changed lines of the file:
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@@
 <part name="GND15" library="SparkFun-Aesthetics" deviceset="GND" device=""/>
 <part name="SUPPLY13" library="SparkFun-Aesthetics" deviceset="5V" device=""/>
-<part name="R19" library="adafruit" deviceset="R-US_" device="0207/10" value="100 kOhm"/>
+<part name="R18" library="adafruit" deviceset="R-US_" device="0207/10" value="100 kOhm"/>
 <part name="C10" library="adafruit" deviceset="CPOL-US" device="E2.5-5" value="0.1 uF"/>
 <part name="GND16" library="SparkFun-Aesthetics" deviceset="GND" device=""/>
@@
 <instance part="GND15" gate="1" x="134.62" y="43.18"/>
 <instance part="SUPPLY13" gate="G$1" x="177.8" y="71.12"/>
-<instance part="R19" gate="G$1" x="154.94" y="53.34"/>
+<instance part="R18" gate="G$1" x="154.94" y="53.34"/>
 <instance part="C10" gate="G$1" x="33.02" y="81.28"/>
 <instance part="GND16" gate="1" x="33.02" y="71.12"/>
@@
 <pinref part="SUPPLY13" gate="G$1" pin="5V"/>
 <wire x1="177.8" y1="53.34" x2="177.8" y2="71.12" width="0.1524" layer="91"/>
-<pinref part="R19" gate="G$1" pin="2"/>
+<pinref part="R18" gate="G$1" pin="2"/>
 <wire x1="160.02" y1="53.34" x2="177.8" y2="53.34" width="0.1524" layer="91"/>
 </segment>
@@
 <wire x1="129.54" y1="63.5" x2="142.24" y2="63.5" width="0.1524" layer="91"/>
 <wire x1="142.24" y1="63.5" x2="142.24" y2="53.34" width="0.1524" layer="91"/>
-<pinref part="R19" gate="G$1" pin="1"/>
+<pinref part="R18" gate="G$1" pin="1"/>
 <wire x1="142.24" y1="53.34" x2="149.86" y2="53.34" width="0.1524" layer="91"/>
 </segment>
