File: Final/Final_bk.brd (EAGLE design)
At the start: 144.4 x 39.4 mm, 27 parts, among them IC1 MCP73871, J1 POWER_JACKPTH, U1 TPS2561DRCT, U2 TPS61030PWPR

Commit message: wired final solar
Parts:
- moved THERM 15.2 mm to (36.8, 17.8)
- moved R6 3.81 mm to (36.8, 14.0), turned to 0 degrees
- moved R7 3.81 mm to (36.8, 10.2), turned to 0 degrees
- moved R9 3.81 mm to (36.8, 6.35), turned to 0 degrees
- moved R10 3.81 mm to (36.8, 2.54)
- moved PWR 1.27 mm to (26.7, 35.6), turned to 270 degrees
- moved C1 1.27 mm to (21.6, 8.89)
- moved C2 1.27 mm to (3.81, 14.0)
- moved CHRG 1.27 mm to (26.7, 27.9), turned to 270 degrees
- moved DONE 1.27 mm to (26.7, 20.3), turned to 270 degrees
- moved J1 1.27 mm to (-1.27, 22.9)
- turned C3 to 0 degrees
- turned C4 to 0 degrees
- turned R5 to 0 degrees
Connections:
- new net N$14: BATT.2, J1.GND
- net GND: no longer BATT.2, J1.GND
- net N$9: now also C2.+, D1.C, U3.VBUS1; no longer DONE.K, IC1.7
- net VCC: no longer C2.+, D1.C, U3.VBUS1
