File: Final/Final.brd (EAGLE design)
At the start: 100 x 80 mm, 27 parts, among them IC1 MCP73871, J1 POWER_JACKPTH, U1 TPS2561DRCT, U2 TPS61030PWPR

Commit message: wired final solar
Parts:
- moved R10 172.6 mm to (34.3, 44.5), turned to 180 degrees
- moved R9 166.7 mm to (34.3, 40.6), turned to 180 degrees
- moved C3 165.3 mm to (16.5, 43.2)
- moved C4 161.8 mm to (3.81, 43.2)
- moved BATT 158.5 mm to (5.71, 35.6), turned to 90 degrees
- moved R7 158.0 mm to (34.3, 36.8), turned to 180 degrees
- moved U1 157.1 mm to (-67.3, 24.1)
- moved R6 152.9 mm to (34.3, 33.0), turned to 180 degrees
- moved R5 148.1 mm to (34.3, 29.2), turned to 180 degrees
- moved R4 143.7 mm to (34.3, 25.4), turned to 180 degrees
- moved CHRG 136.2 mm to (38.1, 8.89), turned to 270 degrees
- moved R3 131.9 mm to (34.3, 21.6), turned to 180 degrees
- moved DONE 130.7 mm to (30.5, 8.89), turned to 270 degrees
- moved R2 129.8 mm to (34.3, 17.8), turned to 180 degrees
- moved R1 128.2 mm to (34.3, 14.0), turned to 180 degrees
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Other:
- board size 100 x 80 mm -> 172.4 x 47 mm

Commit message: wired up solar board
Parts:
- FRAME1: value FRAME-LETTER -> FRAME-LEDGER
- moved U1 132.2 mm to (64.8, 19.1)
- moved U$1 125.0 mm to (101.6, 21.6), turned to 180 degrees
- moved TPS2513 114.6 mm to (86.4, 34.3)
- moved U2 108.4 mm to (72.4, 44.5)
Connections:
- net N$16 renamed V_BATT
Routing:
- net GND: track 0.00 -> 158.0 mm
- net VCC: track 0.00 -> 113.4 mm
- net N$13: track 0.00 -> 86.6 mm
- net N$10: track 0.00 -> 36.5 mm
- net N$3: track 0.00 -> 36.1 mm
- net N$2: track 0.00 -> 33.2 mm, vias 0 -> 1
- net N$12: track 0.00 -> 30.5 mm, vias 0 -> 1
- net N$9: track 0.00 -> 29.8 mm
- net N$14: track 0.00 -> 27.9 mm
- net N$7: track 0.00 -> 21.2 mm
- net N$6: track 0.00 -> 12.0 mm
- net V_BATT: track 0.00 -> 9.46 mm, vias 0 -> 1
- net N$11: track 0.00 -> 7.29 mm, vias 0 -> 1
- net N$1: track 0.00 -> 6.77 mm
- net N$4: track 0.00 -> 6.35 mm
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Other:
- board size 172.4 x 47 mm -> 111.4 x 81.3 mm
