File: Final/Final.brd (EAGLE design)
At the start: 58.1 x 81.3 mm, 47 parts, among them IC1 MCP73871, J1 POWER_JACKPTH, U1 TPS2561DRCT, U2 TPS61030PWPR

Commit message: Made even more tweeks to the design
Parts:
- U3: value (none) -> USB-MICROB; device SparkFun-Connectors:USB-AB-MICRO-SMD_V03 -> SparkFun-Connectors:USB-MICROB
- moved U3 0.64 mm to (2.54, 22.9), turned to 270 degrees
Connections:
- net GND: now also U3.GND, U3.MT1, U3.MT2; no longer U3.GND1
- net VCC: now also U3.VBUS; no longer U3.VBUS1
Routing:
- net GND: track 373.4 -> 383.6 mm
- net N$2: track 33.2 -> 29.6 mm
- net VCC: track 114.7 -> 114.1 mm
Other:
- board text added: "V2 Prototype"
- board text added: "http://cutnop.github.io/Solar-USB-charger/"
- board text removed: "http://cutnop.github.io/ Solar-USB-charger/"
Changed lines of the file:
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@@
 <wire x1="58.09" y1="81.27" x2="0" y2="81.27" width="0" layer="20"/>
 <wire x1="0" y1="81.27" x2="0" y2="0" width="0" layer="20"/>
-<text x="45.72" y="15.24" size="1.778" layer="25" rot="R90">Solar Cell Phone Charger</text>
-<text x="49.53" y="40.64" size="1.778" layer="25" rot="R270">http://cutnop.github.io/
-Solar-USB-charger/</text>
+<text x="45.72" y="29.21" size="1.27" layer="25" rot="R270" align="center">Solar Cell Phone Charger</text>
+<text x="53.34" y="29.21" size="1.27" layer="25" rot="R90" align="center">http://cutnop.github.io/Solar-USB-charger/</text>
+<text x="48.26" y="29.21" size="1.27" layer="25" rot="R90" align="center">V2 Prototype</text>
 </plain>
 <attributes>
@@
 </class>
 </classes>
-<designrules name="default">
+<designrules name="LaenPCBOrder">
 <description language="de">&lt;b&gt;EAGLE Design Rules&lt;/b&gt;
 &lt;p&gt;
@@
 Einstellungen hier und speichern die Design Rules unter
 einem neuen Namen ab.</description>
-<description language="en">&lt;b&gt;EAGLE Design Rules&lt;/b&gt;
+<description language="en">&lt;b&gt;Laen's PCB Order Design Rules&lt;/b&gt;
 &lt;p&gt;
-The default Design Rules have been set to cover
-a wide range of applications. Your particular design
-may have different requirements, so please make the
-necessary adjustments and save your customized
-design rules under a new name.</description>
+Please make sure your boards conform to these design rules.</description>
 <param name="layerSetup" value="(1*16)"/>
-<param name="mtCopper" value="0.035mm 0.035mm 0.035mm 0.035mm 0.035mm 0.035mm 0.035mm 0.035mm 0.035mm 0.035mm 0.035mm 0.035mm 0.035mm 0.035mm 0.035mm 0.035mm"/>
-<param name="mtIsolate" value="1.5mm 0.15mm 0.2mm 0.15mm 0.2mm 0.15mm 0.2mm 0.15mm 0.2mm 0.15mm 0.2mm 0.15mm 0.2mm 0.15mm 0.2mm"/>
-<param name="mdWireWire" value="8mil"/>
-<param name="mdWirePad" value="8mil"/>
-<param name="mdWireVia" value="8mil"/>
-<param name="mdPadPad" value="8mil"/>
-<param name="mdPadVia" value="8mil"/>
-<param name="mdViaVia" value="8mil"/>
-<param name="mdSmdPad" value="8mil"/>
-<param name="mdSmdVia" value="8mil"/>
-<param name="mdSmdSmd" value="8mil"/>
+<param name="mtCopper" value="0.0356mm 0.0356mm 0.0356mm 0.0356mm 0.0356mm 0.0356mm 0.0356mm 0.0356mm 0.0356mm 0.0356mm 0.0356mm 0.0356mm 0.0356mm 0.0356mm 0.0356mm 0.0356mm"/>
+<param name="mtIsolate" value="1.5011mm 0.1499mm 0.2007mm 0.1499mm 0.2007mm 0.1499mm 0.2007mm 0.1499mm 0.2007mm 0.1499mm 0.2007mm 0.1499mm 0.2007mm 0.1499mm 0.2007mm"/>
+<param name="mdWireWire" value="6mil"/>
+<param name="mdWirePad" value="6mil"/>
+<param name="mdWireVia" value="6mil"/>
+<param name="mdPadPad" value="6mil"/>
+<param name="mdPadVia" value="6mil"/>
+<param name="mdViaVia" value="6mil"/>
+<param name="mdSmdPad" value="6mil"/>
+<param name="mdSmdVia" value="6mil"/>
+<param name="mdSmdSmd" value="6mil"/>
 <param name="mdViaViaSameLayer" value="8mil"/>
 <param name="mnLayersViaInSmd" value="2"/>
-<param name="mdCopperDimension" value="40mil"/>
-<param name="mdDrill" value="8mil"/>
+<param name="mdCopperDimension" value="15mil"/>
+<param name="mdDrill" value="6mil"/>
 <param name="mdSmdStop" value="0mil"/>
-<param name="msWidth" value="10mil"/>
-<param name="msDrill" value="24mil"/>
-<param name="msMicroVia" value="9.99mm"/>
+<param name="msWidth" value="6mil"/>
+<param name="msDrill" value="13mil"/>
+<param name="msMicroVia" value="13mil"/>
 <param name="msBlindViaRatio" value="0.5"/>
 <param name="rvPadTop" value="0.25"/>
@@
 <param name="rvMicroViaOuter" value="0.25"/>
 <param name="rvMicroViaInner" value="0.25"/>
-<param name="rlMinPadTop" value="10mil"/>
+<param name="rlMinPadTop" value="7mil"/>
 <param name="rlMaxPadTop" value="20mil"/>
-<param name="rlMinPadInner" value="10mil"/>
+<param name="rlMinPadInner" value="7mil"/>
 <param name="rlMaxPadInner" value="20mil"/>
-<param name="rlMinPadBottom" value="10mil"/>
+<param name="rlMinPadBottom" value="7mil"/>
 <param name="rlMaxPadBottom" value="20mil"/>
-<param name="rlMinViaOuter" value="8mil"/>
+<param name="rlMinViaOuter" value="7mil"/>
 <param name="rlMaxViaOuter" value="20mil"/>
-<param name="rlMinViaInner" value="8mil"/>
+<param name="rlMinViaInner" value="7mil"/>
 <param name="rlMaxViaInner" value="20mil"/>
 <param name="rlMinMicroViaOuter" value="4mil"/>
@@
 <param name="mvStopFrame" value="1"/>
 <param name="mvCreamFrame" value="0"/>
-<param name="mlMinStopFrame" value="4mil"/>
-<param name="mlMaxStopFrame" value="4mil"/>
+<param name="mlMinStopFrame" value="3mil"/>
+<param name="mlMaxStopFrame" value="3mil"/>
 <param name="mlMinCreamFrame" value="0mil"/>
 <param name="mlMaxCreamFrame" value="0mil"/>
@@
 <attribute name="OC_FARNELL" value="-" x="21.59" y="68.58" size="1.778" layer="27" display="off"/>
 </element>
-<element name="U3" library="SparkFun-Connectors" package="USB-AB-MICRO-SMD_V03" value="" x="1.905" y="22.86">
-<attribute name="PROD_ID" value="CONN-11794" x="1.905" y="22.86" size="1.778" layer="27" display="off"/>
+<element name="U3" library="SparkFun-Connectors" package="USB-MICROB" value="USB-MICROB" x="2.54" y="22.86" rot="R270">
+<attribute name="PROD_ID" value="CONN-09505" x="2.54" y="22.86" size="1.778" layer="27" rot="R270" display="off"/>
 </element>
 <element name="C5" library="adafruit" package="E2,5-5" value="10 uF" x="3.81" y="49.53"/>
@@
 <contactref element="C1" pad="-"/>
 <contactref element="C2" pad="-"/>
-<contactref element="U3" pad="GND1"/>
 <contactref element="R5" pad="1"/>
 <contactref element="R6" pad="1"/>
@@
 <wire x1="13.97" y1="45.72" x2="15.24" y2="45.72" width="0.254" layer="1"/>
 <wire x1="15.24" y1="45.72" x2="17.78" y2="43.18" width="0.254" layer="1"/>
-<wire x1="4.605" y1="21.56" x2="6.38" y2="21.56" width="0.254" layer="1"/>
 <wire x1="6.38" y1="21.56" x2="7.62" y2="20.32" width="0.254" layer="1"/>
 <wire x1="7.62" y1="20.32" x2="7.62" y2="17.78" width="0.254" layer="1"/>
 <wire x1="7.62" y1="17.78" x2="5.08" y2="17.78" width="0.254" layer="1"/>
-<wire x1="5.08" y1="17.78" x2="1.27" y2="13.97" width="0.254" layer="1"/>
+<wire x1="5.08" y1="17.78" x2="4.28625" y2="16.98625" width="0.254" layer="1"/>
+<wire x1="4.28625" y1="16.98625" x2="1.27" y2="13.97" width="0.254" layer="1"/>
 <wire x1="1.27" y1="13.97" x2="1.35" y2="13.97" width="0.254" layer="1"/>
 <wire x1="1.35" y1="13.97" x2="7.7" y2="7.62" width="0.254" layer="1"/>
@@
 <wire x1="57.2262" y1="7.62" x2="57.2262" y2="47.0916" width="0.254" layer="1"/>
 <wire x1="57.2262" y1="47.0916" x2="49.5173" y2="47.0027" width="0.254" layer="1"/>
+<wire x1="4.28625" y1="16.98625" x2="3.81" y2="17.4625" width="0.1524" layer="1"/>
+<wire x1="3.81" y1="17.4625" x2="2.54" y2="18.7325" width="0.1524" layer="1"/>
+<wire x1="3.81" y1="25.24125" x2="2.54" y2="26.51125" width="0.1524" layer="1"/>
+<wire x1="3.81" y1="17.4625" x2="3.81" y2="25.24125" width="0.1524" layer="1"/>
+<contactref element="U3" pad="MT1"/>
+<contactref element="U3" pad="MT2"/>
+<contactref element="U3" pad="GND"/>
+<wire x1="2.54" y1="26.51125" x2="2.54" y2="26.86" width="0" layer="19" extent="1-1"/>
+<wire x1="2.54" y1="18.86" x2="2.54" y2="18.7325" width="0" layer="19" extent="1-1"/>
+<wire x1="5.19" y1="21.56" x2="6.38" y2="21.56" width="0" layer="19" extent="1-1"/>
 </signal>
 <signal name="VCC">
@@
 <contactref element="C1" pad="+"/>
 <contactref element="C2" pad="+"/>
-<contactref element="U3" pad="VBUS1"/>
+<contactref element="U3" pad="VBUS"/>
 <contactref element="IC1" pad="17"/>
 <contactref element="IC1" pad="9"/>
@@
 <wire x1="10.16" y1="29.21" x2="10.16" y2="24.13" width="0.254" layer="16"/>
 <wire x1="10.16" y1="24.13" x2="11.43" y2="22.86" width="0.254" layer="16"/>
-<wire x1="4.605" y1="24.16" x2="6.35" y2="24.16" width="0.254" layer="1"/>
+<wire x1="5.19" y1="24.16" x2="6.35" y2="24.16" width="0.254" layer="1"/>
 <wire x1="6.35" y1="24.16" x2="10.13" y2="24.16" width="0.254" layer="1"/>
 <wire x1="10.13" y1="24.16" x2="11.43" y2="22.86" width="0.254" layer="1"/>
@@
 <wire x1="29.21" y1="29.21" x2="35.56" y2="29.21" width="0.254" layer="1"/>
 <wire x1="35.56" y1="29.21" x2="39.37" y2="25.4" width="0.254" layer="1"/>
-<wire x1="19.59" y1="36.06" x2="18.55" y2="36.06" width="0.254" layer="1"/>
-<wire x1="18.55" y1="36.06" x2="17.78" y2="36.83" width="0.254" layer="1"/>
-<via x="17.78" y="36.83" extent="1-16" drill="0.6"/>
-<wire x1="17.78" y1="36.83" x2="17.78" y2="35.56" width="0.254" layer="16"/>
-<wire x1="17.78" y1="35.56" x2="16.51" y2="34.29" width="0.254" layer="16"/>
-<wire x1="16.51" y1="34.29" x2="16.51" y2="31.75" width="0.254" layer="16"/>
-<wire x1="16.51" y1="31.75" x2="19.05" y2="29.21" width="0.254" layer="16"/>
-<wire x1="19.05" y1="29.21" x2="29.21" y2="29.21" width="0.254" layer="16"/>
+<wire x1="19.59" y1="36.06" x2="18.57375" y2="36.06" width="0.254" layer="1"/>
+<wire x1="18.57375" y1="36.06" x2="18.55" y2="36.06" width="0.254" layer="1"/>
+<wire x1="18.57375" y1="36.195" x2="18.57375" y2="36.06" width="0.1524" layer="1"/>
+<wire x1="17.4625" y1="35.08375" x2="18.57375" y2="36.195" width="0.1524" layer="16"/>
+<wire x1="17.4625" y1="33.49625" x2="17.4625" y2="35.08375" width="0.1524" layer="16"/>
+<wire x1="21.74875" y1="29.21" x2="17.4625" y2="33.49625" width="0.1524" layer="16"/>
+<wire x1="29.21" y1="29.21" x2="21.74875" y2="29.21" width="0.1524" layer="16"/>
+<wire x1="18.57375" y1="36.03625" x2="18.57375" y2="36.06" width="0.1524" layer="1"/>
+<via x="18.57375" y="36.195" extent="1-16" drill="0.3302"/>
 </signal>
 <signal name="N$4">
@@
 <wire x1="15.3162" y1="42.9768" x2="16.4592" y2="41.8338" width="0.254" layer="1"/>
 <wire x1="15.3162" y1="42.9768" x2="15.24" y2="43.18" width="0.254" layer="1"/>
-</signal>
-<signal name="N$8">
-<via x="17.78" y="36.83" extent="1-16" drill="0.6"/>
 </signal>
 <signal name="N$18">
@@
 </board>
 </drawing>
-<compatibility>
-<note version="6.3" minversion="6.2.2" severity="warning">
-Since Version 6.2.2 text objects can contain more than one line,
-which will not be processed correctly with this version.
-</note>
-</compatibility>
 </eagle>

Commit message: more tweeks
Parts:
- renumbered R19 to R18
Other:
- board text added: "http://cutnop.github.io /Solar-USB-charger/"
- board text removed: "http://cutnop.github.io/Solar-USB-charger/"
Changed lines of the file:
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@@
 <wire x1="58.09" y1="81.27" x2="0" y2="81.27" width="0" layer="20"/>
 <wire x1="0" y1="81.27" x2="0" y2="0" width="0" layer="20"/>
-<text x="45.72" y="29.21" size="1.27" layer="25" rot="R270" align="center">Solar Cell Phone Charger</text>
-<text x="53.34" y="29.21" size="1.27" layer="25" rot="R90" align="center">http://cutnop.github.io/Solar-USB-charger/</text>
-<text x="48.26" y="29.21" size="1.27" layer="25" rot="R90" align="center">V2 Prototype</text>
+<text x="44.45" y="29.21" size="1.27" layer="25" rot="R270" align="center">Solar Cell Phone Charger</text>
+<text x="46.99" y="29.21" size="1.27" layer="25" rot="R90" align="center">V2 Prototype</text>
+<text x="53.34" y="29.21" size="1.27" layer="25" rot="R90" align="center">http://cutnop.github.io
+/Solar-USB-charger/</text>
 </plain>
 <attributes>
@@
 <element name="LOW" library="adafruit" package="LED5MM" value="" x="45.72" y="8.89" rot="R270"/>
 <element name="R17" library="adafruit" package="0207/10" value="24.9 kOhm" x="50.8" y="58.42"/>
-<element name="R19" library="adafruit" package="0207/10" value="100 kOhm" x="50.8" y="54.61"/>
+<element name="R18" library="adafruit" package="0207/10" value="100 kOhm" x="50.8" y="54.61"/>
 <element name="C10" library="adafruit" package="E2,5-5" value="0.1 uF" x="52.07" y="49.53"/>
 <element name="C11" library="adafruit" package="E2,5-5" value="150 uF" x="45.72" y="49.53"/>
@@
 <wire x1="24.6888" y1="69.0372" x2="24.511" y2="68.9102" width="0.254" layer="1"/>
 <wire x1="21.717" y1="49.6062" x2="21.59" y2="49.53" width="0.254" layer="1"/>
-<contactref element="R19" pad="2"/>
+<contactref element="R18" pad="2"/>
 <contactref element="C10" pad="+"/>
 <contactref element="TPS2513" pad="5"/>
@@
 <signal name="N$26">
 <contactref element="U1" pad="10"/>
-<contactref element="R19" pad="1"/>
+<contactref element="R18" pad="1"/>
 <wire x1="40.005" y1="59.436" x2="37.0332" y2="59.436" width="0.254" layer="1"/>
 <wire x1="40.4622" y1="59.8932" x2="40.005" y2="59.436" width="0.254" layer="1"/>
@@
 </board>
 </drawing>
+<compatibility>
+<note version="6.3" minversion="6.2.2" severity="warning">
+Since Version 6.2.2 text objects can contain more than one line,
+which will not be processed correctly with this version.
+</note>
+</compatibility>
 </eagle>
